File: board/atmega32u4bb.brd (EAGLE design)
At the start: 33 x 12.2 mm, 17 parts, among them Q1 16 MHz

Commit message: Board updated! Looks ok.
Parts:
- S1: device glowboard:KMR211G_SWITCH -> blinkyboard:GLOWBOARD_KMR211G_SWITCH
- U$1: value SMARTPRJ_ATMEGA32U4-XUMU -> ARDUINO_LEONARDO-REV3B_SMARTPRJ_ATMEGA32U4-XUMU; device Arduino_Leonardo-REV3b:SMARTPRJ_QFN44ML7X7 -> blinkyboard:ARDUINO_LEONARDO-REV3B_SMARTPRJ_QFN44ML7X7
- U$3: value PAD_CONNECTION -> GLOWBOARD_PAD_CONNECTION; device glowboard:PAD_CONNECTION -> blinkyboard:GLOWBOARD_PAD_CONNECTION
- U$4: value ICSP -> GLOWBOARD_ICSP; device glowboard:ICSP_PADS -> blinkyboard:GLOWBOARD_ICSP_PADS
Routing:
- net N$11: track 0.00 -> 15.5 mm
- net GND: track 98.0 -> 96.7 mm
- net VCC: track 70.1 -> 71.3 mm
