File: board/BlinkyBoard.sch (EAGLE design)
At the start: 17 parts, among them Q1 16 MHz

Commit message: Add silk, make ground trace wider, rename to BlinkyBoard
Parts:
- added U$2: GLOWBOARD_USB_TEST_PADS, blinkyboard:GLOWBOARD_USB_TEST_PADS
- R1, R2: device adafruit:R-US_R0805 -> blinkyboard:RESISTOR_0805
Connections:
- removed net N$2: R2.1, U$6.D+
- removed net N$5: R1.1, U$6.D-
- new net D+_IN: R2.1, U$2.D+, U$6.D+
- new net D-_IN: R1.1, U$2.D-, U$6.D-
Changed lines of the file:
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@@
 </classes>
 <parts>
-<part name="R1" library="adafruit" deviceset="R-US_" device="R0805" value="22"/>
-<part name="R2" library="adafruit" deviceset="R-US_" device="R0805" value="22"/>
+<part name="R1" library="blinkyboard" deviceset="RESISTOR_0805" device="" value="22"/>
+<part name="R2" library="blinkyboard" deviceset="RESISTOR_0805" device="" value="22"/>
 <part name="GND1" library="supply1" deviceset="GND" device=""/>
 <part name="C1" library="adafruit" deviceset="C-US" device="C0805K" value="0.1uF"/>
@@
 <part name="U$6" library="blinkyboard" deviceset="GLOWBOARD_MINI_USB" device=""/>
 <part name="C5" library="adafruit" deviceset="C-US" device="C0805K" value="0uF (DNC)"/>
+<part name="U$2" library="blinkyboard" deviceset="GLOWBOARD_USB_TEST_PADS" device=""/>
 </parts>
 <sheets>
@@
 <instance part="U$6" gate="G$1" x="-50.8" y="35.56"/>
 <instance part="C5" gate="G$1" x="132.08" y="71.12"/>
+<instance part="U$2" gate="G$1" x="-15.24" y="43.18"/>
 </instances>
 <busses>
@@
 </segment>
 </net>
-<net name="N$2" class="0">
+<net name="D+_IN" class="0">
 <segment>
 <pinref part="R2" gate="G$1" pin="1"/>
-<wire x1="-15.24" y1="35.56" x2="-38.1" y2="35.56" width="0.1524" layer="91"/>
+<wire x1="-15.24" y1="35.56" x2="-27.94" y2="35.56" width="0.1524" layer="91"/>
+<wire x1="-27.94" y1="35.56" x2="-38.1" y2="35.56" width="0.1524" layer="91"/>
 <wire x1="-38.1" y1="35.56" x2="-40.64" y2="33.02" width="0.1524" layer="91"/>
 <pinref part="U$6" gate="G$1" pin="D+"/>
-</segment>
-</net>
-<net name="N$5" class="0">
+<pinref part="U$2" gate="G$1" pin="D+"/>
+<wire x1="-22.86" y1="48.26" x2="-27.94" y2="48.26" width="0.1524" layer="91"/>
+<wire x1="-27.94" y1="48.26" x2="-27.94" y2="35.56" width="0.1524" layer="91"/>
+<junction x="-27.94" y="35.56"/>
+</segment>
+</net>
+<net name="D-_IN" class="0">
 <segment>
 <pinref part="R1" gate="G$1" pin="1"/>
-<wire x1="-5.08" y1="38.1" x2="-40.64" y2="38.1" width="0.1524" layer="91"/>
+<wire x1="-5.08" y1="38.1" x2="-25.4" y2="38.1" width="0.1524" layer="91"/>
 <pinref part="U$6" gate="G$1" pin="D-"/>
-</segment>
-</net>
+<pinref part="U$2" gate="G$1" pin="D-"/>
+<wire x1="-25.4" y1="38.1" x2="-40.64" y2="38.1" width="0.1524" layer="91"/>
+<wire x1="-22.86" y1="45.72" x2="-25.4" y2="45.72" width="0.1524" layer="91"/>
+<wire x1="-25.4" y1="45.72" x2="-25.4" y2="38.1" width="0.1524" layer="91"/>
+<junction x="-25.4" y="38.1"/>
+</segment>
+</net>

Commit message: Hopefully Rev A!!
Parts:
- C1: value 0.1uF -> .1uF
Connections:
- net N$3 renamed D-
- net N$4 renamed D+
- net N$1: now also U$1.(ADC5/TMS)PF5; no longer U$1.(ADC0)PF0
Other:
- moved on the sheet: U$3
Changed lines of the file:
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@@
 <part name="R2" library="blinkyboard" deviceset="RESISTOR_0805" device="" value="22"/>
 <part name="GND1" library="supply1" deviceset="GND" device=""/>
-<part name="C1" library="adafruit" deviceset="C-US" device="C0805K" value="0.1uF"/>
+<part name="C1" library="adafruit" deviceset="C-US" device="C0805K" value=".1uF"/>
 <part name="GND3" library="supply1" deviceset="GND" device=""/>
 <part name="GND6" library="supply1" deviceset="GND" device=""/>
@@
 </segment>
 </net>
-<net name="N$3" class="0">
+<net name="D-" class="0">
 <segment>
 <pinref part="R1" gate="G$1" pin="2"/>
@@
 </segment>
 </net>
-<net name="N$4" class="0">
+<net name="D+" class="0">
 <segment>
 <pinref part="U$1" gate="G$1" pin="D+"/>
@@
 <net name="N$1" class="0">
 <segment>
-<pinref part="U$1" gate="G$1" pin="(ADC0)PF0"/>
-<wire x1="96.52" y1="5.08" x2="104.14" y2="5.08" width="0.1524" layer="91"/>
-<wire x1="104.14" y1="5.08" x2="104.14" y2="7.62" width="0.1524" layer="91"/>
 <pinref part="U$5" gate="G$1" pin="1"/>
 <wire x1="104.14" y1="7.62" x2="111.76" y2="7.62" width="0.1524" layer="91"/>
-</segment>
-</net>
+<wire x1="104.14" y1="7.62" x2="104.14" y2="17.78" width="0.1524" layer="91"/>
+<pinref part="U$1" gate="G$1" pin="(ADC5/TMS)PF5"/>
+<wire x1="104.14" y1="17.78" x2="96.52" y2="17.78" width="0.1524" layer="91"/>
+</segment>
+</net>

Commit message: Replace mini USB footprint with Micro USB, swap in 0603 components and smaller crystal, add ground plane to backside
Parts:
- removed C5: 0uF (DNC), adafruit:C-USC0805K
- C1: value .1uF -> 1uF; device adafruit:C-USC0805K -> adafruit:C-USC0603
- C2, C3, C4, C6, C7, C8: device adafruit:C-USC0805K -> adafruit:C-USC0603
- Q1: device glowboard:ABMM2 -> blinkiverse:CRYSTAL
- R1, R2: device blinkyboard:RESISTOR_0805 -> adafruit:R-US_R0603
- U$1: device blinkyboard:ARDUINO_LEONARDO-REV3B_SMARTPRJ_ATMEGA32U4-XUMU -> blinkiverse:ARDUINO_LEONARDO-REV3B_SMARTPRJ_ATMEGA32U4-XUMU
- U$6: value GLOWBOARD_MINI_USB -> USB-MICROB; device blinkyboard:GLOWBOARD_MINI_USB -> SparkFun:USB-MICROB
Connections:
- net N$10: no longer C5.2
- net RST: no longer C5.1
Other:
- moved on the sheet: C2, C3, U$1
